Commit message: turning wheel

File: src/lekiwi/config/lekiwi.ros2_control.xacro (robot description, xacro)
@@ -59,4 +59,26 @@
         <!-- <state_interface name="velocity"/> -->
       </joint>
+      <!-- WHEEL JOINTS (Motor IDs 7-9) -->
+      <joint name="left_wheel_drive">
+        <command_interface name="position" />
+        <state_interface name="position">
+          <param name="initial_value">${initial_positions['left_wheel_drive']}</param>
+        </state_interface>
+        <!-- <state_interface name="velocity"/> -->
+      </joint>
+      <joint name="rear_wheel_drive">
+        <command_interface name="position" />
+        <state_interface name="position">
+          <param name="initial_value">${initial_positions['rear_wheel_drive']}</param>
+        </state_interface>
+        <!-- <state_interface name="velocity"/> -->
+      </joint>
+      <joint name="right_wheel_drive">
+        <command_interface name="position" />
+        <state_interface name="position">
+          <param name="initial_value">${initial_positions['right_wheel_drive']}</param>
+        </state_interface>
+        <!-- <state_interface name="velocity"/> -->
+      </joint>
     </ros2_control>
   </xacro:macro>

Commit message: add omniwheel controller

File: src/lekiwi/config/lekiwi.ros2_control.xacro (robot description, xacro)
@@ -59,25 +59,25 @@
         <!-- <state_interface name="velocity"/> -->
       </joint>
-      <!-- WHEEL JOINTS (Motor IDs 7-9) -->
+      <!-- WHEEL JOINTS (Motor IDs 7-9) - Use velocity control -->
       <joint name="left_wheel_drive">
-        <command_interface name="position" />
+        <command_interface name="velocity" />
         <state_interface name="position">
           <param name="initial_value">${initial_positions['left_wheel_drive']}</param>
         </state_interface>
-        <!-- <state_interface name="velocity"/> -->
+        <state_interface name="velocity" />
       </joint>
       <joint name="rear_wheel_drive">
-        <command_interface name="position" />
+        <command_interface name="velocity" />
         <state_interface name="position">
           <param name="initial_value">${initial_positions['rear_wheel_drive']}</param>
         </state_interface>
-        <!-- <state_interface name="velocity"/> -->
+        <state_interface name="velocity" />
       </joint>
       <joint name="right_wheel_drive">
-        <command_interface name="position" />
+        <command_interface name="velocity" />
         <state_interface name="position">
           <param name="initial_value">${initial_positions['right_wheel_drive']}</param>
         </state_interface>
-        <!-- <state_interface name="velocity"/> -->
+        <state_interface name="velocity" />
       </joint>
     </ros2_control>

File: src/lekiwi/config/lekiwi.urdf.xacro (robot description, xacro)
@@ -2,12 +2,21 @@
 <robot xmlns:xacro="http://www.ros.org/wiki/xacro" name="lekiwi">
     <xacro:arg name="initial_positions_file" default="initial_positions.yaml" />
-    <xacro:arg name="use_fake_hardware" default="false"/>
+    <xacro:arg name="use_fake_hardware" default="false" />
     <!-- Import lekiwi urdf file -->
     <xacro:include filename="$(find lekiwi)/urdf/lekiwi_complete.urdf" />
     <!-- Import control_xacro -->
     <xacro:include filename="lekiwi.ros2_control.xacro" />
+    <!-- Add base_footprint as the root frame with proper orientation -->
+    <!-- This aligns the coordinate system: X=forward, Y=left, Z=up -->
+    <link name="base_footprint" />
+    <joint name="base_footprint_joint" type="fixed">
+        <parent link="base_footprint" />
+        <child link="base_link" />
+        <!-- Rotate 90° counterclockwise around Z-axis to align coordinate frames -->
+        <origin xyz="0 0 0" rpy="0 0 -1.5708" />
+    </joint>
     <xacro:lekiwi_ros2_control
         name="SO100ARM"
         initial_positions_file="$(arg initial_positions_file)"
-        use_fake_hardware="$(arg use_fake_hardware)"/>
+        use_fake_hardware="$(arg use_fake_hardware)" />
 </robot>
