Commit message: arm control in ik

File: src/lekiwi/config/lekiwi.urdf.xacro (robot description, xacro)
@@ -2,7 +2,7 @@
 <robot xmlns:xacro="http://www.ros.org/wiki/xacro" name="lekiwi">
     <xacro:arg name="initial_positions_file" default="initial_positions.yaml" />
-    <xacro:arg name="use_fake_hardware" default="false" />
+    <xacro:arg name="use_fake_hardware" default="false"/>
     <!-- Import lekiwi urdf file -->
-    <xacro:include filename="$(find lekiwi)/urdf/lekiwi_5dof.urdf" />
+    <xacro:include filename="$(find lekiwi)/urdf/lekiwi_complete.urdf" />
     <!-- Import control_xacro -->
     <xacro:include filename="lekiwi.ros2_control.xacro" />
@@ -10,4 +10,4 @@
         name="SO100ARM"
         initial_positions_file="$(arg initial_positions_file)"
-        use_fake_hardware="$(arg use_fake_hardware)" />
+        use_fake_hardware="$(arg use_fake_hardware)"/>
 </robot>

File: src/lekiwi/urdf/lekiwi_5dof.urdf (robot description, URDF)
Before this commit: robot lekiwi, 8 links, 7 joints
Links:
- removed link Base
- added link Base_08q-v1, mass 0.193184127927598; collision mesh filename=file://$(find lekiwi)/models/lekiwi_5dof/meshes/Base.STL; visual mesh filename=file://$(find lekiwi)/models/lekiwi_5dof/meshes/Base.STL
Joints:
- joint Shoulder_Rotation: parent Base -> Base_08q-v1
- joint base_link_joint: child Base -> Base_08q-v1

Commit message: add nav2

File: src/lekiwi/config/lekiwi.urdf.xacro (robot description, xacro)
@@ -3,6 +3,6 @@
     <xacro:arg name="initial_positions_file" default="initial_positions.yaml" />
     <xacro:arg name="use_fake_hardware" default="false" />
-    <!-- Import lekiwi urdf file -->
-    <xacro:include filename="$(find lekiwi)/urdf/lekiwi_complete.urdf" />
+    <!-- Import lekiwi mobile base urdf file (includes proper base frame connections) -->
+    <xacro:include filename="$(find lekiwi)/urdf/lekiwi_mobile_base.urdf" />
     <!-- Import control_xacro -->
     <xacro:include filename="lekiwi.ros2_control.xacro" />
@@ -12,6 +12,6 @@
     <joint name="base_footprint_joint" type="fixed">
         <parent link="base_footprint" />
-        <child link="base_link" />
-        <!-- Rotate 90° counterclockwise around Z-axis to align coordinate frames -->
+        <child link="mobile_base_link" />
+        <!-- Apply 90-degree rotation to align coordinate frames: X=forward, Y=left -->
         <origin xyz="0 0 0" rpy="0 0 -1.5708" />
     </joint>

Commit message: clean up repository

File: src/lekiwi/config/lekiwi.urdf.xacro (robot description, xacro)
@@ -4,5 +4,5 @@
     <xacro:arg name="use_fake_hardware" default="false" />
     <!-- Import lekiwi mobile base urdf file (includes proper base frame connections) -->
-    <xacro:include filename="$(find lekiwi)/urdf/lekiwi_mobile_base.urdf" />
+    <xacro:include filename="$(find lekiwi)/urdf/lekiwi_complete.urdf" />
     <!-- Import control_xacro -->
     <xacro:include filename="lekiwi.ros2_control.xacro" />
@@ -12,5 +12,5 @@
     <joint name="base_footprint_joint" type="fixed">
         <parent link="base_footprint" />
-        <child link="mobile_base_link" />
+        <child link="base_link" />
         <!-- Apply 90-degree rotation to align coordinate frames: X=forward, Y=left -->
         <origin xyz="0 0 0" rpy="0 0 -1.5708" />
